Commit message: added gazebo plugin model

File: src/journey/urdf/quadrotor_base.urdf.xacro (robot description, xacro)
@@ -35,20 +35,19 @@
     </joint>
     <gazebo reference="base_link">
-      <turnGravityOff>false</turnGravityOff>
-      <sensor type="contact" name="/${sim_name}/collision">
-        <always_on>true</always_on>
-        <update_rate>10</update_rate>
-        <contact>
-          <collision>base_link_collision</collision>
-        </contact>
-        <plugin name="bumper_plugin" filename="libgazebo_ros_bumper.so">
-          <bumperTopicName>${sim_name}/crash_sensor</bumperTopicName>
-          <frameName>${sim_name}/crash_sensor</frameName>
-        </plugin>
-      </sensor>
+        <sensor name="mode_c_radar" type="logical_camera">
+            <visualize>true</visualize>
+            <always_on>true</always_on>
+            <update_rate>10</update_rate>
+            <plugin name="mode_c_radar" filename="libModeCRadarPlugin.so">
+                <position_noise>
+                    <noise>
+                        <type>gaussian</type>
+                        <mean>0.0</mean>
+                        <stddev>0.001</stddev>
+                    </noise>
+                </position_noise>
+            </plugin>
+        </sensor>
     </gazebo>
-    <!-- Radar sensor -->
-    <xacro:include filename="$(find cvg_sim_gazebo)/urdf/sensors/radar_sensor.urdf.xacro" />
-    <xacro:radar/>
     <!-- Gazebo Plugins -->
     <quadrotor_plugins/>

File: src/journey/urdf/quadrotor_sensors.urdf.xacro (robot description, xacro)
@@ -10,9 +10,4 @@
     <!-- Instantiate quadrotor_base_macro once (has no parameters atm) -->
     <quadrotor_base_macro sim_name="ardrone"/>
-    <!-- Sonar height sensor -->
-    <xacro:include filename="$(find cvg_sim_gazebo)/urdf/sensors/sonar_sensor.urdf.xacro" />
-    <xacro:sonar_sensor name="sonar" parent="base_link" ros_topic="sonar_height" update_rate="10" min_range="0.01" max_range="3.0" field_of_view="${40*M_PI/180}" ray_count="3">
-      <origin xyz="-0.15 0.0 0.0" rpy="0 ${90*M_PI/180} 0"/>
-    </xacro:sonar_sensor>
     <!-- Hokuyo UTM-30LX mounted upside down below the quadrotor body
     <xacro:include filename="$(find cvg_sim_gazebo)/urdf/sensors/hokuyo_utm30lx.urdf.xacro" />
@@ -20,7 +15,3 @@
       <origin xyz="0.0 0.0 0.08" rpy="${M_PI} 0 0"/>
     </xacro:hokuyo_utm30lx>-->
-    <!-- The following two cameras should be united to one! -->
-    <!-- Forward facing camera -->
-    <xacro:include filename="$(find journey)/urdf/sensors/radar_sensor.urdf.xacro" />
-    <xacro:radar/>
 </robot>

File: src/journey/urdf/sensors/radar_sensor.urdf.xacro (robot description, xacro)
@@ -4,91 +4,40 @@
 xmlns:xacro="http://ros.org/wiki/xacro">
 <xacro:macro name="radar">
-    <!-- <link name="rad_link">
-      <inertial>
-        <mass value="0.001" />
-        <origin xyz="0 0 0" rpy="0 0 0" />
-        <inertia ixx="0.000000017" ixy="0" ixz="0" iyy="0.000000017" iyz="0" izz="0.000000017" />
-      </inertial>
-      <visual>
-        <origin xyz="0 0 0" rpy="0 0 0" />
-        <geometry>
-          <box size="0.01 0.01 0.01" />
-         <mesh filename="package://cvg_sim_gazebo/meshes/kinect_camera/kinect_camera_simple.dae"/>
-        </geometry>
-      </visual>
-      <collision>
-        <origin xyz="0 0 0" rpy="0 0 0" />
-        <geometry>
-          <box size="0.01 0.01 0.01" />
-        </geometry>
-      </collision>
-    </link> -->
-    <plugin name="mode_c_radar" filename="libModeCRadarPlugin.so">
-        <robotNamespace>radar</robotNamespace>
-        <position_noise>
-          <noise>
-            <type>gaussian</type>
-            <mean>0.0</mean>
-            <stddev>0.001</stddev>
-          </noise>
-        </position_noise>
-        <known_model_types>
-          <type>iris</type>
-          <type>delta_wing</type>
-        </known_model_types>
-      </plugin>
-      <link name="radar_mount">
-        <gravity>false</gravity>
+     <link name="rad_link">
+        <collision>
+            <origin xyz="0.2 0 0.2" rpy="0 0 0"/>
+            <geometry>
+                <box size="0.05 0.05 0.05"/>
+            </geometry>
+        </collision>
+        <visual>
+            <origin xyz="0.2 0 0.2" rpy="0 0 0"/>
+            <geometry>
+                <box size="0.05 0.05 0.05"/>
+                <material name="blue"/>
+                <!-- <mesh filename="package://husky_description/meshes/accessories/dummy_camera.dae" /> -->
+            </geometry>
+        </visual>
         <inertial>
-          <mass value="0.001" />
-          <origin xyz="0 0 0" rpy="0 0 0" />
-          <inertia ixx="0.000000017" ixy="0" ixz="0" iyy="0.000000017" iyz="0" izz="0.000000017" />
+            <mass value="1e-5" />
+            <origin xyz="0.2 0 0.2" rpy="0 0 0"/>
+            <inertia ixx="1e-6" ixy="0" ixz="0" iyy="1e-6" iyz="0" izz="1e-6" />
         </inertial>
-        <!-- <collision name="collision">
-          <pose>0 0.02 0 0 0 -1.5708</pose>
-          <geometry>
-            <mesh>
-              <uri>model://logical_camera/meshes/camera.dae</uri>
-            </mesh>
-          </geometry>
-        </collision>
-        <visual name="visual">
-          <pose>0 0.02 0 0 0 -1.5708</pose>
-          <geometry>
-            <mesh>
-              <uri>model://logical_camera/meshes/camera.dae</uri>
-            </mesh>
-          </geometry>
-        </visual> -->
-        <sensor name="logical_camera" type="logical_camera">
-          <logical_camera>
-            <near>0.2</near>
-            <far>2.0</far>
-            <horizontal_fov>1.04719755</horizontal_fov>
-            <aspect_ratio>1.778</aspect_ratio>
-          </logical_camera>
-          <visualize>true</visualize>
-          <always_on>true</always_on>
-          <update_rate>10</update_rate>
-        </sensor>
-      </link>
-      <joint name='radar_mount_joint' type='fixed'>
+    </link>
+    <joint name="radar_joint" type="fixed">
+        <axis xyz="0.2 0 0.2" />
+        <origin xyz="0.2 0 0.2" rpy="0 0 0"/>
         <parent link="base_link"/>
-	      <child link="radar_mount"/>
-      </joint>
-    <!-- <gazebo reference="rad_link">
+        <child link="rad_link"/>
+    </joint>
+    <gazebo reference="rad_link">
         <sensor name="radar" type="logical_camera">
-            <logical_camera>
-            <near>0.55</near>
-            <far>2.5</far>
-            <horizontal_fov>1.05</horizontal_fov>
-            <aspect_ratio>1.8</aspect_ratio>
-          </logical_camera>
-          <visualize>true</visualize>
-          <always_on>true</always_on>
-          <update_rate>10</update_rate>
+            <visualize>true</visualize>
+            <always_on>true</always_on>
+            <update_rate>10</update_rate>
             <plugin name="mode_c_radar" filename="libModeCRadarPlugin.so">
                 <robotNamespace>radar</robotNamespace>
-                <radar_topic_ros>radar_data</radar_topic_ros>
+                <radar_sensor_frameid>rad_link</radar_sensor_frameid>
+                <radar_topic_ros>radar_topic</radar_topic_ros>
                 <position_noise>
                     <noise>
@@ -104,5 +53,5 @@
             </plugin>
         </sensor>
-    </gazebo> -->
+    </gazebo>
 </xacro:macro>
  </robot>

Commit message: tried to add the radar to the drone, not complete

File: src/journey/urdf/quadrotor_base.urdf.xacro (robot description, xacro)
@@ -34,20 +34,40 @@
       <child link="dummy_link"/>
     </joint>
-    <gazebo reference="base_link">
-        <sensor name="mode_c_radar" type="logical_camera">
-            <visualize>true</visualize>
-            <always_on>true</always_on>
-            <update_rate>10</update_rate>
-            <plugin name="mode_c_radar" filename="libModeCRadarPlugin.so">
-                <position_noise>
-                    <noise>
-                        <type>gaussian</type>
-                        <mean>0.0</mean>
-                        <stddev>0.001</stddev>
-                    </noise>
-                </position_noise>
-            </plugin>
-        </sensor>
+<joint name = "radar" type = "fixed">
+    <parent link = "base_link"/>
+    <child link="dummy_link"/>
+<gazebo reference="radar_link">
+<sensor name="sensor_ray" type="ray">
+    <visualize>true</visualize>
+    <pose>0.1 0.0 0.0 -1.57079632679 -1.57079632679 0.0</pose>
+    <ray>
+      <scan>
+        <horizontal>
+          <samples>100</samples>
+          <min_angle>-0.523599</min_angle>
+          <max_angle>0.523599</max_angle>
+        </horizontal>
+        <vertical>
+          <samples>16</samples>
+          <min_angle>-0.261799</min_angle>
+          <max_angle>0.261799</max_angle>
+        </vertical>
+      </scan>
+      <range>
+        <min>0.05</min>
+        <max>80.0</max>
+      </range>
+    </ray>
+    <plugin name="plugin_1" filename="libgazebo_ros_block_laser.so">
+      <gaussianNoise>0.00</gaussianNoise>
+      <hokuyoMinIntensity>1</hokuyoMinIntensity>
+      <alwaysOn>true</alwaysOn>
+      <updateRate>5</updateRate>
+      <topicName>radar</topicName>
+      <frameName>base_link</frameName>
+    </plugin>
+  </sensor>
     </gazebo>
+</joint>
     <!-- Gazebo Plugins -->
     <quadrotor_plugins/>

File: src/journey/urdf/quadrotor_sensors.urdf.xacro (robot description, xacro)
@@ -10,8 +10,3 @@
     <!-- Instantiate quadrotor_base_macro once (has no parameters atm) -->
     <quadrotor_base_macro sim_name="ardrone"/>
-    <!-- Hokuyo UTM-30LX mounted upside down below the quadrotor body
-    <xacro:include filename="$(find cvg_sim_gazebo)/urdf/sensors/hokuyo_utm30lx.urdf.xacro" />
-    <xacro:hokuyo_utm30lx name="laser0" parent="base_link" ros_topic="scan" update_rate="40" ray_count="1081" min_angle="135" max_angle="-135">
-      <origin xyz="0.0 0.0 0.08" rpy="${M_PI} 0 0"/>
-    </xacro:hokuyo_utm30lx>-->
 </robot>

File: src/journey/urdf/sensors/radar_sensor.urdf.xacro (robot description, xacro)
@@ -25,5 +25,5 @@
         </inertial>
     </link>
-    <joint name="radar_joint" type="fixed">
+    <joint name="sensor_ray" type="ray">
         <axis xyz="0.2 0 0.2" />
         <origin xyz="0.2 0 0.2" rpy="0 0 0"/>
@@ -32,25 +32,34 @@
     </joint>
     <gazebo reference="rad_link">
-        <sensor name="radar" type="logical_camera">
-            <visualize>true</visualize>
-            <always_on>true</always_on>
-            <update_rate>10</update_rate>
-            <plugin name="mode_c_radar" filename="libModeCRadarPlugin.so">
-                <robotNamespace>radar</robotNamespace>
-                <radar_sensor_frameid>rad_link</radar_sensor_frameid>
-                <radar_topic_ros>radar_topic</radar_topic_ros>
-                <position_noise>
-                    <noise>
-                        <type>gaussian</type>
-                        <mean>0.0</mean>
-                        <stddev>0.001</stddev>
-                    </noise>
-                </position_noise>
-                <known_model_types>
-                    <type>husky</type>
-                    <type>delta_wing</type>
-                </known_model_types>
-            </plugin>
-        </sensor>
+<sensor name="sensor_ray" type="ray">
+    <visualize>true</visualize>
+    <pose>0.1 0.0 0.0 -1.57079632679 -1.57079632679 0.0</pose>
+    <ray>
+      <scan>
+        <horizontal>
+          <samples>100</samples>
+          <min_angle>-0.523599</min_angle>
+          <max_angle>0.523599</max_angle>
+        </horizontal>
+        <vertical>
+          <samples>16</samples>
+          <min_angle>-0.261799</min_angle>
+          <max_angle>0.261799</max_angle>
+        </vertical>
+      </scan>
+      <range>
+        <min>0.05</min>
+        <max>80.0</max>
+      </range>
+    </ray>
+    <plugin name="plugin_1" filename="libgazebo_ros_block_laser.so">
+      <gaussianNoise>0.00</gaussianNoise>
+      <hokuyoMinIntensity>1</hokuyoMinIntensity>
+      <alwaysOn>true</alwaysOn>
+      <updateRate>5</updateRate>
+      <topicName>radar</topicName>
+      <frameName>base_link</frameName>
+    </plugin>
+  </sensor>
     </gazebo>
 </xacro:macro>

Commit message: added radar to drone

File: src/journey/urdf/quadrotor_base.urdf.xacro (robot description, xacro)
@@ -34,40 +34,4 @@
       <child link="dummy_link"/>
     </joint>
-<joint name = "radar" type = "fixed">
-    <parent link = "base_link"/>
-    <child link="dummy_link"/>
-<gazebo reference="radar_link">
-<sensor name="sensor_ray" type="ray">
-    <visualize>true</visualize>
-    <pose>0.1 0.0 0.0 -1.57079632679 -1.57079632679 0.0</pose>
-    <ray>
-      <scan>
-        <horizontal>
-          <samples>100</samples>
-          <min_angle>-0.523599</min_angle>
-          <max_angle>0.523599</max_angle>
-        </horizontal>
-        <vertical>
-          <samples>16</samples>
-          <min_angle>-0.261799</min_angle>
-          <max_angle>0.261799</max_angle>
-        </vertical>
-      </scan>
-      <range>
-        <min>0.05</min>
-        <max>80.0</max>
-      </range>
-    </ray>
-    <plugin name="plugin_1" filename="libgazebo_ros_block_laser.so">
-      <gaussianNoise>0.00</gaussianNoise>
-      <hokuyoMinIntensity>1</hokuyoMinIntensity>
-      <alwaysOn>true</alwaysOn>
-      <updateRate>5</updateRate>
-      <topicName>radar</topicName>
-      <frameName>base_link</frameName>
-    </plugin>
-  </sensor>
-    </gazebo>
-</joint>
     <!-- Gazebo Plugins -->
     <quadrotor_plugins/>

File: src/journey/urdf/quadrotor_sensors.urdf.xacro (robot description, xacro)
@@ -10,3 +10,10 @@
     <!-- Instantiate quadrotor_base_macro once (has no parameters atm) -->
     <quadrotor_base_macro sim_name="ardrone"/>
+    <!-- Sonar height sensor -->
+    <xacro:include filename="$(find cvg_sim_gazebo)/urdf/sensors/sonar_sensor.urdf.xacro" />
+    <xacro:sonar_sensor name="sonar" parent="base_link" ros_topic="sonar_height" update_rate="10" min_range="0.01" max_range="3.0" field_of_view="${40*M_PI/180}" ray_count="3">
+      <origin xyz="-0.15 0.0 0.0" rpy="0 ${90*M_PI/180} 0"/>
+    </xacro:sonar_sensor>
+    <xacro:include filename="$(find journey)/urdf/sensors/radar_sensor.urdf.xacro" />
+    <xacro:radar/>
 </robot>

File: src/journey/urdf/sensors/radar_sensor.urdf.xacro (robot description, xacro)
@@ -25,5 +25,5 @@
         </inertial>
     </link>
-    <joint name="sensor_ray" type="ray">
+    <joint name="sensor_ray" type="fixed">
         <axis xyz="0.2 0 0.2" />
         <origin xyz="0.2 0 0.2" rpy="0 0 0"/>
@@ -32,34 +32,34 @@
     </joint>
     <gazebo reference="rad_link">
-<sensor name="sensor_ray" type="ray">
-    <visualize>true</visualize>
-    <pose>0.1 0.0 0.0 -1.57079632679 -1.57079632679 0.0</pose>
-    <ray>
-      <scan>
-        <horizontal>
-          <samples>100</samples>
-          <min_angle>-0.523599</min_angle>
-          <max_angle>0.523599</max_angle>
-        </horizontal>
-        <vertical>
-          <samples>16</samples>
-          <min_angle>-0.261799</min_angle>
-          <max_angle>0.261799</max_angle>
-        </vertical>
-      </scan>
-      <range>
-        <min>0.05</min>
-        <max>80.0</max>
-      </range>
-    </ray>
-    <plugin name="plugin_1" filename="libgazebo_ros_block_laser.so">
-      <gaussianNoise>0.00</gaussianNoise>
-      <hokuyoMinIntensity>1</hokuyoMinIntensity>
-      <alwaysOn>true</alwaysOn>
-      <updateRate>5</updateRate>
-      <topicName>radar</topicName>
-      <frameName>base_link</frameName>
-    </plugin>
-  </sensor>
+      <sensor name="sensor_ray" type="ray">
+          <visualize>true</visualize>
+          <pose>0.1 0.0 0.0 -1.57079632679 -1.57079632679 0.0</pose>
+          <ray>
+            <scan>
+              <horizontal>
+                <samples>100</samples>
+                <min_angle>-0.523599</min_angle>
+                <max_angle>0.523599</max_angle>
+              </horizontal>
+              <vertical>
+                <samples>16</samples>
+                <min_angle>-0.261799</min_angle>
+                <max_angle>0.261799</max_angle>
+              </vertical>
+            </scan>
+            <range>
+              <min>0.05</min>
+              <max>80.0</max>
+            </range>
+          </ray>
+          <plugin name="plugin_1" filename="libgazebo_ros_block_laser.so">
+            <gaussianNoise>0.00</gaussianNoise>
+            <hokuyoMinIntensity>1</hokuyoMinIntensity>
+            <alwaysOn>true</alwaysOn>
+            <updateRate>5</updateRate>
+            <topicName>radar</topicName>
+            <frameName>base_link</frameName>
+          </plugin>
+        </sensor>
     </gazebo>
 </xacro:macro>
