Commit message: update drone model

File: src/journey/urdf/sensors/radar_sensor.urdf.xacro (robot description, xacro)
@@ -11,11 +11,17 @@
             </geometry>
         </collision>
-        <visual>
-            <origin xyz="0.2 0 0.2" rpy="0 0 0"/>
-            <geometry>
-                <box size="0.05 0.05 0.05"/>
-                <material name="blue"/>
-                <!-- <mesh filename="package://husky_description/meshes/accessories/dummy_camera.dae" /> -->
-            </geometry>
+        <visual name="AWR1642BOOST_visual">
+          <geometry>
+            <box>
+              <size> 0.2 0.4 0.01 </size>
+            </box>
+          </geometry>
+        </visual>
+        <visual name="DCA1000EVM_visual">
+          <geometry>
+            <box>
+              <size> 0.2 0.4 0.01 </size>
+            </box>
+          </geometry>
         </visual>
         <inertial>

Commit message: added the sensor to the model, need to add the DCA too

File: src/journey/urdf/sensors/radar_sensor.urdf.xacro (robot description, xacro)
@@ -5,29 +5,21 @@
 <xacro:macro name="radar">
      <link name="rad_link">
-        <collision>
-            <origin xyz="0.2 0 0.2" rpy="0 0 0"/>
-            <geometry>
-                <box size="0.05 0.05 0.05"/>
-            </geometry>
-        </collision>
-        <visual name="AWR1642BOOST_visual">
-          <geometry>
-            <box>
-              <size> 0.2 0.4 0.01 </size>
-            </box>
-          </geometry>
-        </visual>
-        <visual name="DCA1000EVM_visual">
-          <geometry>
-            <box>
-              <size> 0.2 0.4 0.01 </size>
-            </box>
-          </geometry>
-        </visual>
-        <inertial>
-            <mass value="1e-5" />
-            <origin xyz="0.2 0 0.2" rpy="0 0 0"/>
-            <inertia ixx="1e-6" ixy="0" ixz="0" iyy="1e-6" iyz="0" izz="1e-6" />
-        </inertial>
+    <!-- Offset the base by half the lenght of the cylinder -->
+      <inertial>
+      <mass value= "1.2"/>
+      <inertia ixx = "0.001087473" iyy="0.001087473" izz ="0.001087473" ixy="0" ixz="0" iyz="0"/>
+    </inertial>
+    <collision name="AWR1642BOOST_collision">
+      <geometry>
+        <box size="0.2 0.4 0.01"/>
+      </geometry>
+    </collision>
+    <!-- The visual is mostly a copy of the collision -->
+    <visual name="AWR1642BOOST_visual">
+		<origin xyz="0 0 0" rpy="1.5708 0 1.5708"/>
+      <geometry>
+        <box size="0.2 0.4 0.01"/>
+      </geometry>
+    </visual>
     </link>
     <joint name="sensor_ray" type="fixed">
@@ -40,5 +32,5 @@
       <sensor name="sensor_ray" type="ray">
           <visualize>true</visualize>
-          <pose>0.1 0.0 0.0 -1.57079632679 -1.57079632679 0.0</pose>
+		  <pose> 0 0 0 -1.57079632679 -1.57079632679 0.0 </pose>
           <ray>
             <scan>
@@ -55,5 +47,5 @@
             </scan>
             <range>
-              <min>0.05</min>
+              <min>0.15</min>
               <max>80.0</max>
             </range>
@@ -70,3 +62,3 @@
     </gazebo>
 </xacro:macro>
- </robot>
+</robot>

Commit message: fixed the radar sensor to be added to the drone module. Still need to update inertia and size to be more accurate

File: src/journey/urdf/sensors/radar_sensor.urdf.xacro (robot description, xacro)
@@ -4,61 +4,83 @@
 xmlns:xacro="http://ros.org/wiki/xacro">
 <xacro:macro name="radar">
-     <link name="rad_link">
-    <!-- Offset the base by half the lenght of the cylinder -->
-      <inertial>
-      <mass value= "1.2"/>
-      <inertia ixx = "0.001087473" iyy="0.001087473" izz ="0.001087473" ixy="0" ixz="0" iyz="0"/>
+<link name="rad_link">
+    <!-- Physics of the AWR1642 -->
+	<inertial>
+      	<mass value= "1.2"/>
+      	<inertia ixx = "0.001087473" iyy="0.001087473" izz ="0.001087473" ixy="0" ixz="0" iyz="0"/>
     </inertial>
     <collision name="AWR1642BOOST_collision">
-      <geometry>
-        <box size="0.2 0.4 0.01"/>
-      </geometry>
+      	<geometry>
+        	<box size="0.2 0.4 0.01"/>
+      	</geometry>
     </collision>
-    <!-- The visual is mostly a copy of the collision -->
+    <!-- The visual part of the boost -->
     <visual name="AWR1642BOOST_visual">
 		<origin xyz="0 0 0" rpy="1.5708 0 1.5708"/>
-      <geometry>
-        <box size="0.2 0.4 0.01"/>
-      </geometry>
+     	<geometry>
+        	<box size="0.2 0.4 0.01"/>
+      	</geometry>
     </visual>
-    </link>
-    <joint name="sensor_ray" type="fixed">
-        <axis xyz="0.2 0 0.2" />
-        <origin xyz="0.2 0 0.2" rpy="0 0 0"/>
-        <parent link="base_link"/>
-        <child link="rad_link"/>
-    </joint>
-    <gazebo reference="rad_link">
-      <sensor name="sensor_ray" type="ray">
-          <visualize>true</visualize>
-		  <pose> 0 0 0 -1.57079632679 -1.57079632679 0.0 </pose>
-          <ray>
-            <scan>
-              <horizontal>
-                <samples>100</samples>
-                <min_angle>-0.523599</min_angle>
-                <max_angle>0.523599</max_angle>
-              </horizontal>
-              <vertical>
-                <samples>16</samples>
-                <min_angle>-0.261799</min_angle>
-                <max_angle>0.261799</max_angle>
-              </vertical>
-            </scan>
-            <range>
-              <min>0.15</min>
-              <max>80.0</max>
-            </range>
-          </ray>
-          <plugin name="plugin_1" filename="libgazebo_ros_block_laser.so">
-            <gaussianNoise>0.00</gaussianNoise>
-            <hokuyoMinIntensity>1</hokuyoMinIntensity>
-            <alwaysOn>true</alwaysOn>
-            <updateRate>5</updateRate>
-            <topicName>radar</topicName>
-            <frameName>base_link</frameName>
-          </plugin>
-        </sensor>
-    </gazebo>
+	<!-- Physics for the DCA1000 component -->
+   	<inertial>
+   		<mass value="0.1"/>
+    	<inertia ixx="0.000090623" iyy="0.000090623" izz="0.000090623" ixy="0" ixz="0" iyz="0"/>
+   	</inertial>
+    <collision name="DCA1000EVM_collision">
+      	<geometry>
+        	<box size="0.2 0.4 0.01"/>
+      	</geometry>
+    </collision>
+	<!-- Visuals of the DCA1000EVM -->
+    <visual name="DCA1000EVM_visual">
+		<origin xyz="-0.05 0 0" rpy="1.5708 0 1.5708"/>
+    	<geometry>
+       		<box size = "0.2 0.4 0.01"/>
+    	</geometry>
+    </visual>
+</link>
+<!-- setting up a joint for the sensor -->
+<joint name="sensor_ray" type="fixed">
+	<axis xyz="0.2 0 0.2" />
+	<origin xyz="0.2 0 0.2" rpy="0 0 0"/>
+	<parent link="base_link"/>
+	<child link="rad_link"/>
+</joint>
+<!-- set up the gazebo reference -->
+<gazebo reference="rad_link">
+	<sensor name="sensor_ray" type="ray">
+		<visualize>true</visualize>
+		<pose> 0 0 0 -1.57079632679 -1.57079632679 0.0 </pose>
+		<ray>
+			<scan>
+				<!-- to adjust the horizontal and verticle samples -->
+				<horizontal>
+					<samples>100</samples>
+					<min_angle>-0.523599</min_angle>
+					<max_angle>0.523599</max_angle>
+				</horizontal>
+				<vertical>
+					<samples>16</samples>
+					<min_angle>-0.261799</min_angle>
+					<max_angle>0.261799</max_angle>
+				</vertical>
+			</scan>
+			<!-- to adjust the min/max hit distance for each laser -->
+			<range>
+				<min>0.15</min>
+				<max>80.0</max>
+			</range>
+		</ray>
+		<!-- to control the plugin and how much noise is on it -->
+		<plugin name="plugin_1" filename="libgazebo_ros_block_laser.so">
+			<gaussianNoise>0.00</gaussianNoise>
+			<hokuyoMinIntensity>1</hokuyoMinIntensity>
+			<alwaysOn>true</alwaysOn>
+			<updateRate>5</updateRate>
+			<topicName>radar</topicName>
+			<frameName>base_link</frameName>
+		</plugin>
+	</sensor>
+</gazebo>
 </xacro:macro>
 </robot>

Commit message: trying to fix the inertia on the drone

File: src/journey/urdf/sensors/radar_sensor.urdf.xacro (robot description, xacro)
@@ -7,15 +7,15 @@
     <!-- Physics of the AWR1642 -->
 	<inertial>
-      	<mass value= "1.2"/>
+      	<mass value= "0.25"/>
       	<inertia ixx = "0.001087473" iyy="0.001087473" izz ="0.001087473" ixy="0" ixz="0" iyz="0"/>
     </inertial>
     <collision name="AWR1642BOOST_collision">
       	<geometry>
-        	<box size="0.2 0.4 0.01"/>
+        	<box size="0.1 0.2 0.01"/>
       	</geometry>
     </collision>
     <!-- The visual part of the boost -->
     <visual name="AWR1642BOOST_visual">
-		<origin xyz="0 0 0" rpy="1.5708 0 1.5708"/>
+		<origin xyz="-0.14 0 0" rpy="1.5708 0 1.5708"/>
      	<geometry>
         	<box size="0.2 0.4 0.01"/>
@@ -24,15 +24,15 @@
 	<!-- Physics for the DCA1000 component -->
    	<inertial>
-   		<mass value="0.1"/>
+   		<mass value="0.25"/>
     	<inertia ixx="0.000090623" iyy="0.000090623" izz="0.000090623" ixy="0" ixz="0" iyz="0"/>
    	</inertial>
     <collision name="DCA1000EVM_collision">
       	<geometry>
-        	<box size="0.2 0.4 0.01"/>
+        	<box size="0.1 0.2 0.01"/>
       	</geometry>
     </collision>
 	<!-- Visuals of the DCA1000EVM -->
     <visual name="DCA1000EVM_visual">
-		<origin xyz="-0.05 0 0" rpy="1.5708 0 1.5708"/>
+		<origin xyz="-0.19 0 0" rpy="1.5708 0 1.5708"/>
     	<geometry>
        		<box size = "0.2 0.4 0.01"/>

Commit message: fixed visual size

File: src/journey/urdf/sensors/radar_sensor.urdf.xacro (robot description, xacro)
@@ -19,5 +19,5 @@
 		<origin xyz="-0.14 0 0" rpy="1.5708 0 1.5708"/>
      	<geometry>
-        	<box size="0.2 0.4 0.01"/>
+        	<box size="0.1 0.2 0.01"/>
       	</geometry>
     </visual>
@@ -36,5 +36,5 @@
 		<origin xyz="-0.19 0 0" rpy="1.5708 0 1.5708"/>
     	<geometry>
-       		<box size = "0.2 0.4 0.01"/>
+       		<box size = "0.1 0.2 0.01"/>
     	</geometry>
     </visual>

Commit message: set mass to 0 to stop weird drifting affect

File: src/journey/urdf/sensors/radar_sensor.urdf.xacro (robot description, xacro)
@@ -7,5 +7,5 @@
     <!-- Physics of the AWR1642 -->
 	<inertial>
-      	<mass value= "0.25"/>
+      	<mass value= "0.0"/>
       	<inertia ixx = "0.001087473" iyy="0.001087473" izz ="0.001087473" ixy="0" ixz="0" iyz="0"/>
     </inertial>
@@ -24,5 +24,5 @@
 	<!-- Physics for the DCA1000 component -->
    	<inertial>
-   		<mass value="0.25"/>
+   		<mass value="0.0"/>
     	<inertia ixx="0.000090623" iyy="0.000090623" izz="0.000090623" ixy="0" ixz="0" iyz="0"/>
    	</inertial>
